File: at820_tiga.kicad_pcb (KiCad board)
At the start: 2 copper layers, 93.5 x 82.5 mm, 107 parts, among them J1 TEST_MODE, J10 USB, J11 QSPI_SWITCH, J12 Conn_01x03_Pin, J13 Conn_01x03_Pin, J2 SWD, J3 Download, J4 I2C0, J5 UART0, J6 SPI0, J7 Power, J8 Conn_01x04_Pin, J9 UART, SW1 OS102011MS2QN1, SW2 Reset, SW3 Wakeup, SW4 Boot, SW5 Loopback, U1 TS5A23157DGS, U3 CH343P, U4 AMS1117-3.3, U5 MIX2909, Y1 Crystal_GND24

Commit message: v2 done
Parts:
- added Q1: SS8050, Package_TO_SOT_SMD:SOT-23, F.Cu at (129.5, 116.6)
- added Q2: SS8050, Package_TO_SOT_SMD:SOT-23, F.Cu at (128.4, 126.7)
- added R7: 10K, Resistor_SMD:R_0603_1608Metric_Pad0.98x0.95mm_HandSolder, F.Cu at (125.5, 126.9)
- added R8: 10K, Resistor_SMD:R_0603_1608Metric_Pad0.98x0.95mm_HandSolder, F.Cu at (129.6, 122.3)
- C1: value 10uF/NC -> 0.1uF
- C13: value 10uF -> 0.1uF
- D12: footprint Diode_SMD:D_SOD-323 -> Diode_SMD:D_SMA_Handsoldering
- J11: value QSPI_SWITCH -> QSPI
- J3: footprint Connector_PinHeader_2.54mm:PinHeader_1x04_P2.54mm_Vertical -> Connector_PinHeader_2.54mm:PinHeader_1x05_P2.54mm_Vertical
- L1: footprint Inductor_SMD:L_Changjiang_FTC404020S -> Inductor_SMD:L_APV_APH0420
- MK1: value RMic -> RMIC; footprint Capacitor_THT:CP_Radial_D4.0mm_P1.50mm -> Sensor_Audio:POM-2244P-C3310-2-R
- MK2: value LMic -> LMIC; footprint Capacitor_THT:CP_Radial_D4.0mm_P1.50mm -> Sensor_Audio:POM-2244P-C3310-2-R
- R1: value 10K/NC -> 10K
- moved MK2 26.1 mm to (117.5, 58.5)
- moved R24 25.6 mm to (116.2, 69.5)
- moved R27 25.6 mm to (121.2, 69.5)
- moved R25 25.6 mm to (116.2, 65.4)
- moved R26 25.6 mm to (121.2, 65.4)
- moved C35 25.6 mm to (118.7, 67.3)
- moved R21 19.5 mm to (142.0, 69.5)
- moved R20 19.5 mm to (142.0, 65.4)
- moved C31 14.3 mm to (139.3, 67.3)
- moved MK1 12.9 mm to (138.5, 58.5), turned to 0 degrees
- moved R18 9.14 mm to (136.6, 69.5)
- moved R19 9.14 mm to (136.6, 65.4)
- moved R6 7.76 mm to (123.7, 126.9)
- moved SW4 6.80 mm to (156.8, 134.5)
- moved C15 6.80 mm to (156.7, 131.0)
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- renumbered AT820-Tiga to AT820-Tiga-V2, C15 to C14, C14 to C15, R8 to R10, R9 to R11, R10 to R12, R11 to R13, R12 to R14, R13 to R15, R14 to R16, R15 to R17, R16 to R18, R17 to R19, R18 to R20, R19 to R21, R20 to R22, R21 to R23, R22 to R24, R23 to R25, R24 to R26, R25 to R27, R7 to R9, SW4 to SW3, SW3 to SW4
Connections:
- D1 pad 1: +3V3 -> Net-(D1-K)
- D1 pad 2: Net-(D1-A) -> +3V3
- D2 pad 1: +3V3 -> Net-(D2-K)
- D2 pad 2: Net-(D2-A) -> +3V3
- J2 pad 2: /AT_RST -> /AT_SWCLK
- J2 pad 3: /AT_SWCLK -> /AT_SWDIO
- J2 pad 4: /AT_SWDIO -> +3V3
- R4 pad 2: Net-(D1-A) -> Net-(D1-K)
- R5 pad 2: Net-(D2-A) -> Net-(D2-K)
- U3 pad 12: /AT_BOOT -> /CH_DTR
- U3 pad 13: /AT_RST -> /CH_RTS
- U3 pad 4: /CH_UART_RXD -> /CH_UART_TXD
- U3 pad 5: /CH_UART_TXD -> /CH_UART_RXD
Routing:
- net /AT_LMIC_P: track 28.4 -> 59.9 mm, vias 0 -> 1
- net /AT_LMIC_N: track 26.0 -> 57.3 mm, vias 0 -> 1
- net /AT_RST: track 126.0 -> 99.6 mm
- net GND: track 49.8 -> 32.1 mm, vias 91 -> 86
- net VBUS: track 73.4 -> 58.0 mm, vias 7 -> 6
- net /AT_RMIC_N: track 67.5 -> 54.8 mm
- net /AT_GPIO3: track 85.3 -> 96.9 mm
- net Net-(Q1-B): track 0.00 -> 11.5 mm, vias 0 -> 2
- net /CH_RTS: track 0.00 -> 7.95 mm
- net AT_MICBIAS: track 37.3 -> 44.6 mm, vias 3 -> 4
- net /AT_PWM0: track 72.4 -> 77.4 mm
- net Net-(D12-A): track 13.9 -> 8.93 mm
- net /CH_DTR: track 0.00 -> 4.86 mm
- net GNDA: track 50.7 -> 46.4 mm
- net Net-(Q2-B): track 0.00 -> 3.91 mm
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Other:
- board text added: "DIO"
- board text removed: "SWCLK"
- board text removed: "SWDIO"
