File: at820_tiga.kicad_sch (KiCad schematic)
At the start: 36 parts, among them J1 SWD, J13 TEST_MODE, J2 download, J3 I2C, J4 uart0, J5 SPI0, J6 power, J7 Conn_01x04_Pin, SW1 OS102011MS2QN1, SW2 Wakeup Button, SW3 Reset Button, SW6 Boot Button, U2 CH343P, U3 TS5A23157DGS, Y1 Crystal_GND24

Commit message: beta 2, modify board size, add some silkscreen
Parts:
- added D1, D2: LED, LED_SMD:LED_0603_1608Metric_Pad1.05x0.95mm_HandSolder, symbol Device:LED
- added R4, R5: 2K, Resistor_SMD:R_0603_1608Metric_Pad0.98x0.95mm_HandSolder, symbol Device:R_US
- J3: renamed from J2; value download -> Download
- J4: renamed from J3; value I2C -> I2C0
- J5: renamed from J4; value uart0 -> UART0
- J7: renamed from J6; value power -> Power
- SW2: renamed from SW3; value Reset Button -> Reset
- SW3: renamed from SW2; value Wakeup Button -> Wakeup
- SW4: renamed from SW6; value Boot Button -> Boot
- renumbered C13 to C10, C14 to C11, C5 to C12, C6 to C13, C4 to C14, C36 to C15, C7 to C4, C8 to C5, C9 to C6, C10 to C7, C11 to C8, C12 to C9, J13 to J1, J1 to J2, J5 to J6, J7 to J8, R5 to R6, R4 to R7, U3 to U1, U1 to U2, U2 to U3
Connections:
- net +3V3: now also D1.1 (K), D2.1 (K)
- net CH_UART_RXD: now also R4.1
- net CH_UART_TXD: now also R5.1
- new net: D1.2 (A), R4.2
- new net: D2.2 (A), R5.2
Other:
- moved on the sheet: SW1, U1B

Commit message: refactor crystal pcb
Parts:
- Y1: footprint Crystal:Crystal_SMD_3225-4Pin_3.2x2.5mm_HandSoldering -> Crystal:Crystal_SMD_3225-4Pin_3.2x2.5mm
Changed lines of the file:
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@@
 			)
 		)
-		(property "Footprint" "Crystal:Crystal_SMD_3225-4Pin_3.2x2.5mm_HandSoldering"
+		(property "Footprint" "Crystal:Crystal_SMD_3225-4Pin_3.2x2.5mm"
 			(at 41.91 172.72 0)
 			(hide yes)

Commit message: fix ch343p bug and other bugs in sch
Parts:
- added Q1, Q2: SS8050, Package_TO_SOT_SMD:SOT-23, symbol Transistor_BJT:SS8050
- added R26, R27: 10K, Resistor_SMD:R_0603_1608Metric_Pad0.98x0.95mm_HandSolder, symbol Device:R_US
- C1: value 10uF/NC -> 0.1uF
- C13: value 10uF -> 0.1uF
- R1: value 10K/NC -> 10K
Connections:
- net +3V3: now also D1.2 (A), D2.2 (A); no longer D1.1 (K), D2.1 (K)
- net AT_BOOT: now also Q2.3 (C); no longer U3.12 (~{DTR})
- net AT_RST: now also Q1.3 (C); no longer U3.13 (~{RTS})
- net CH_UART_RXD: now also U3.5 (RXD); no longer U3.4 (TXD)
- net CH_UART_TXD: now also U3.4 (TXD); no longer U3.5 (RXD)
- net at R4.2: now also D1.1 (K); no longer D1.2 (A)
- net at R5.2: now also D2.1 (K); no longer D2.2 (A)
- new net: Q1.1 (B), R26.1
- new net: Q2.1 (B), R27.2
- new net CH_DTR: Q2.2 (E), R26.2, U3.12 (~{DTR})
- new net CH_RTS: Q1.2 (E), R27.1, U3.13 (~{RTS})
Other:
- moved on the sheet: C12, C13, C15, D1, D2, J2, J3, J4, J5, J6, J7, J8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

Commit message: v2 done
Parts:
- removed J3: Download, Connector_PinHeader_2.54mm:PinHeader_1x04_P2.54mm_Vertical, symbol Connector:Conn_01x04_Pin
- added J3: Download, Connector_PinHeader_2.54mm:PinHeader_1x05_P2.54mm_Vertical, symbol Connector:Conn_01x05_Pin
- renumbered C15 to C14, C14 to C15, R26 to R7, R27 to R8, R7 to R9, SW4 to SW3, SW3 to SW4
Connections:
- net +3V3: now also J2.4 (Pin_4)
- net AT_BOOT: now also J3.4 (Pin_4)
- net AT_RST: now also J3.5 (Pin_5); no longer J2.2 (Pin_2)
- net AT_SWCLK: now also J2.2 (Pin_2); no longer J2.3 (Pin_3)
- net AT_SWDIO: now also J2.3 (Pin_3); no longer J2.4 (Pin_4)
- net AT_SYS_UART_RXD: now also J3.2 (Pin_2)
- net AT_SYS_UART_TXD: now also J3.3 (Pin_3)
- net GND: now also J3.1 (Pin_1)
Other:
- moved on the sheet: C12, C13, C14, C15, J2, J4, J5, J6, J7, J8, Q1, Q2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
