File: audio.kicad_sch (KiCad schematic)
At the start: 28 parts, among them J11 Conn_01x03_Pin, J12 Conn_01x03_Pin, SW4 MY_SW_DPST, U5 MIX2909

Commit message: beta 2, modify board size, add some silkscreen
Parts:
- L1: value 6.8uH -> 6.8uH PCR0420-6R8-M; footprint Inductor_SMD:L_Sunlord_MWSA0402S -> Inductor_SMD:L_Changjiang_FTC404020S
- SW5: renamed from SW4; value MY_SW_DPST -> Loopback
- renumbered C27 to C28, C28 to C29, C29 to C30, C30 to C31, C31 to C32, C32 to C33, C33 to C34, C34 to C35, C35 to C36, D4 to D12, J11 to J12, J12 to J13, R15 to R16, R16 to R17, R17 to R18, R18 to R19, R19 to R20, R20 to R21, R21 to R22, R22 to R23, R23 to R24, R24 to R25

Commit message: fix ch343p bug and other bugs in sch
Parts:
- D12: footprint Diode_SMD:D_SOD-323 -> Diode_SMD:D_SMA-SMB_Universal_Handsoldering
- L1: footprint Inductor_SMD:L_Changjiang_FTC404020S -> Inductor_SMD:L_APV_APH0420
Changed lines of the file:
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@@
 			)
 		)
-		(property "Footprint" "Inductor_SMD:L_Changjiang_FTC404020S"
+		(property "Footprint" "Inductor_SMD:L_APV_APH0420"
 			(at 40.64 60.96 0)
 			(hide yes)
@@
 			)
 		)
-		(property "Footprint" "Diode_SMD:D_SOD-323"
+		(property "Footprint" "Diode_SMD:D_SMA-SMB_Universal_Handsoldering"
 			(at 63.5 56.515 0)
 			(hide yes)

Commit message: v2 done
Parts:
- D12: footprint Diode_SMD:D_SMA-SMB_Universal_Handsoldering -> Diode_SMD:D_SMA_Handsoldering
- MK1: value Microphone -> RMIC; footprint Capacitor_THT:CP_Radial_D4.0mm_P1.50mm -> Sensor_Audio:POM-2244P-C3310-2-R
- MK2: value Microphone -> LMIC; footprint Capacitor_THT:CP_Radial_D4.0mm_P1.50mm -> Sensor_Audio:POM-2244P-C3310-2-R
- renumbered R16 to R18, R17 to R19, R18 to R20, R19 to R21, R20 to R22, R21 to R23, R22 to R24, R23 to R25, R24 to R26, R25 to R27
Other:
- moved on the sheet: J12
Changed lines of the file:
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@@
 		)
 	)
-	(label "AT_RMIC_N"
-		(at 195.58 123.19 0)
+	(label "PA_OUTP"
+		(at 233.68 38.1 180)
 		(effects
 			(font
 				(size 1.27 1.27)
 			)
-			(justify left bottom)
+			(justify right bottom)
 		)
 	)
-	(label "AT_RMIC_P"
-		(at 195.58 116.84 0)
+	(label "AT_RMIC_N"
+		(at 195.58 123.19 0)
 		(effects
 			(font
@@
 		)
 	)
-	(label "PA_OUTP"
-		(at 207.01 38.1 0)
+	(label "AT_RMIC_P"
+		(at 195.58 116.84 0)
 		(effects
 			(font
@@
 		)
 	)
-	(label "AT_LOUT_P"
-		(at 233.68 38.1 180)
+	(label "PA_EN"
+		(at 81.28 78.74 180)
 		(effects
 			(font
@@
 		)
 	)
-	(label "PA_EN"
-		(at 81.28 78.74 180)
+	(label "AT_LMIC_N"
+		(at 195.58 110.49 0)
 		(effects
 			(font
 				(size 1.27 1.27)
 			)
-			(justify right bottom)
+			(justify left bottom)
 		)
 	)
-	(label "AT_LMIC_N"
-		(at 195.58 110.49 0)
+	(label "AT_LOUT_P"
+		(at 207.01 38.1 0)
 		(effects
 			(font
@@
 		(dnp no)
 		(fields_autoplaced yes)
-		(property "Reference" "#PWR084"
+		(property "Reference" "#PWR085"
 			(at 44.45 124.46 0)
 			(hide yes)
@@
 			(project "at820_tiga"
 				(path "/a8c0f85c-55b6-4da9-ba8c-71a36ed08e24/3b744c5c-59b1-4c52-9315-8adf8de34fd5"
-					(reference "#PWR084")
+					(reference "#PWR085")
 					(unit 1)
 				)
@@
 		(dnp no)
 		(fields_autoplaced yes)
-		(property "Reference" "#PWR087"
+		(property "Reference" "#PWR088"
 			(at 97.79 81.28 0)
 			(hide yes)
@@
 			(project "at820_tiga"
 				(path "/a8c0f85c-55b6-4da9-ba8c-71a36ed08e24/3b744c5c-59b1-4c52-9315-8adf8de34fd5"
-					(reference "#PWR087")
+					(reference "#PWR088")
 					(unit 1)
 				)
@@
 		(dnp no)
 		(fields_autoplaced yes)
-		(property "Reference" "R25"
+		(property "Reference" "R27"
 			(at 127 172.7199 0)
 			(show_name no)
@@
 			(project "at820_tiga"
 				(path "/a8c0f85c-55b6-4da9-ba8c-71a36ed08e24/3b744c5c-59b1-4c52-9315-8adf8de34fd5"
-					(reference "R25")
+					(reference "R27")
 					(unit 1)
 				)
@@
 		(dnp no)
 		(fields_autoplaced yes)
-		(property "Reference" "R20"
+		(property "Reference" "R22"
 			(at 73.66 29.21 90)
 			(show_name no)
@@
 			(project "at820_tiga"
 				(path "/a8c0f85c-55b6-4da9-ba8c-71a36ed08e24/3b744c5c-59b1-4c52-9315-8adf8de34fd5"
-					(reference "R20")
+					(reference "R22")
 					(unit 1)
 				)
@@
 		(dnp no)
 		(fields_autoplaced yes)
-		(property "Reference" "#PWR088"
+		(property "Reference" "#PWR089"
 			(at 124.46 121.92 0)
 			(hide yes)
@@
 			(project "at820_tiga"
 				(path "/a8c0f85c-55b6-4da9-ba8c-71a36ed08e24/3b744c5c-59b1-4c52-9315-8adf8de34fd5"
-					(reference "#PWR088")
+					(reference "#PWR089")
 					(unit 1)
 				)
@@
 		(dnp no)
 		(fields_autoplaced yes)
-		(property "Reference" "R19"
+		(property "Reference" "R21"
 			(at 46.99 175.2599 0)
 			(show_name no)
@@
 			(project "at820_tiga"
 				(path "/a8c0f85c-55b6-4da9-ba8c-71a36ed08e24/3b744c5c-59b1-4c52-9315-8adf8de34fd5"
-					(reference "R19")
+					(reference "R21")
 					(unit 1)
 				)
@@
 		(dnp no)
 		(fields_autoplaced yes)
-		(property "Reference" "#PWR085"
+		(property "Reference" "#PWR086"
 			(at 44.45 190.5 0)
 			(hide yes)
@@
 			(project "at820_tiga"
 				(path "/a8c0f85c-55b6-4da9-ba8c-71a36ed08e24/3b744c5c-59b1-4c52-9315-8adf8de34fd5"
-					(reference "#PWR085")
+					(reference "#PWR086")
 					(unit 1)
 				)
@@
 		(dnp no)
 		(fields_autoplaced yes)
-		(property "Reference" "R16"
+		(property "Reference" "R18"
 			(at 46.99 125.7299 0)
 			(show_name no)
@@
 			(project "at820_tiga"
 				(path "/a8c0f85c-55b6-4da9-ba8c-71a36ed08e24/3b744c5c-59b1-4c52-9315-8adf8de34fd5"
-					(reference "R16")
+					(reference "R18")
 					(unit 1)
 				)
@@
 		(dnp no)
 		(fields_autoplaced yes)
-		(property "Reference" "#PWR082"
+		(property "Reference" "#PWR083"
 			(at 34.29 58.42 0)
 			(hide yes)
@@
 			(project "at820_tiga"
 				(path "/a8c0f85c-55b6-4da9-ba8c-71a36ed08e24/3b744c5c-59b1-4c52-9315-8adf8de34fd5"
-					(reference "#PWR082")
+					(reference "#PWR083")
 					(unit 1)
 				)
@@
 		(dnp no)
 		(fields_autoplaced yes)
-		(property "Reference" "R17"
+		(property "Reference" "R19"
 			(at 46.99 135.8899 0)
 			(show_name no)
@@
 			(project "at820_tiga"
 				(path "/a8c0f85c-55b6-4da9-ba8c-71a36ed08e24/3b744c5c-59b1-4c52-9315-8adf8de34fd5"
-					(reference "R17")
+					(reference "R19")
 					(unit 1)
 				)
@@
 			)
 		)
-		(property "Footprint" "Diode_SMD:D_SMA-SMB_Universal_Handsoldering"
+		(property "Footprint" "Diode_SMD:D_SMA_Handsoldering"
 			(at 63.5 56.515 0)
 			(hide yes)
@@
 		(dnp no)
 		(property "Reference" "MK2"
-			(at 119.888 147.32 0)
+			(at 125.476 147.32 0)
 			(show_name no)
 			(do_not_autoplace no)
@@
 			)
 		)
-		(property "Value" "Microphone"
-			(at 119.888 149.86 0)
+		(property "Value" "LMIC"
+			(at 125.476 149.86 0)
 			(show_name no)
 			(do_not_autoplace no)
@@
 			)
 		)
-		(property "Footprint" "Capacitor_THT:CP_Radial_D4.0mm_P1.50mm"
+		(property "Footprint" "Sensor_Audio:POM-2244P-C3310-2-R"
 			(at 133.35 151.13 90)
 			(hide yes)
@@
 		(dnp no)
 		(fields_autoplaced yes)
-		(property "Reference" "R22"
+		(property "Reference" "R24"
 			(at 127 123.1899 0)
 			(show_name no)
@@
 			(project "at820_tiga"
 				(path "/a8c0f85c-55b6-4da9-ba8c-71a36ed08e24/3b744c5c-59b1-4c52-9315-8adf8de34fd5"
-					(reference "R22")
+					(reference "R24")
 					(unit 1)
 				)
@@
 		(dnp no)
 		(fields_autoplaced yes)
-		(property "Reference" "#PWR091"
+		(property "Reference" "#PWR092"
 			(at 147.32 58.42 0)
 			(hide yes)
@@
 			(project "at820_tiga"
 				(path "/a8c0f85c-55b6-4da9-ba8c-71a36ed08e24/3b744c5c-59b1-4c52-9315-8adf8de34fd5"
-					(reference "#PWR091")
+					(reference "#PWR092")
 					(unit 1)
 				)
@@
 	(symbol
 		(lib_id "Connector:Conn_01x03_Pin")
-		(at 219.71 30.48 270)
+		(at 219.71 30.48 90)
+		(mirror x)
 		(unit 1)
 		(body_style 1)
@@
 		(in_pos_files yes)
 		(dnp no)
-		(fields_autoplaced yes)
 		(property "Reference" "J12"
 			(at 219.71 25.4 90)
@@
 		(dnp no)
 		(fields_autoplaced yes)
-		(property "Reference" "#PWR089"
+		(property "Reference" "#PWR090"
 			(at 124.46 187.96 0)
 			(hide yes)
@@
 			(project "at820_tiga"
 				(path "/a8c0f85c-55b6-4da9-ba8c-71a36ed08e24/3b744c5c-59b1-4c52-9315-8adf8de34fd5"
-					(reference "#PWR089")
+					(reference "#PWR090")
 					(unit 1)
 				)
@@
 		(dnp no)
 		(fields_autoplaced yes)
-		(property "Reference" "R24"
+		(property "Reference" "R26"
 			(at 127 162.5599 0)
 			(show_name no)
@@
 			(project "at820_tiga"
 				(path "/a8c0f85c-55b6-4da9-ba8c-71a36ed08e24/3b744c5c-59b1-4c52-9315-8adf8de34fd5"
-					(reference "R24")
+					(reference "R26")
 					(unit 1)
 				)
@@
 		(dnp no)
 		(fields_autoplaced yes)
-		(property "Reference" "#PWR086"
+		(property "Reference" "#PWR087"
 			(at 76.2 66.04 0)
 			(hide yes)
@@
 			(project "at820_tiga"
 				(path "/a8c0f85c-55b6-4da9-ba8c-71a36ed08e24/3b744c5c-59b1-4c52-9315-8adf8de34fd5"
-					(reference "#PWR086")
+					(reference "#PWR087")
 					(unit 1)
 				)
@@
 		(dnp no)
 		(fields_autoplaced yes)
-		(property "Reference" "#PWR090"
+		(property "Reference" "#PWR091"
 			(at 147.32 38.1 0)
 			(hide yes)
@@
 			(project "at820_tiga"
 				(path "/a8c0f85c-55b6-4da9-ba8c-71a36ed08e24/3b744c5c-59b1-4c52-9315-8adf8de34fd5"
-					(reference "#PWR090")
+					(reference "#PWR091")
 					(unit 1)
 				)
@@
 		(dnp no)
 		(property "Reference" "MK1"
-			(at 39.878 149.86 0)
+			(at 45.72 150.114 0)
 			(show_name no)
 			(do_not_autoplace no)
@@
 			)
 		)
-		(property "Value" "Microphone"
-			(at 39.878 152.4 0)
+		(property "Value" "RMIC"
+			(at 45.72 152.654 0)
 			(show_name no)
 			(do_not_autoplace no)
@@
 			)
 		)
-		(property "Footprint" "Capacitor_THT:CP_Radial_D4.0mm_P1.50mm"
+		(property "Footprint" "Sensor_Audio:POM-2244P-C3310-2-R"
 			(at 53.34 153.67 90)
 			(hide yes)
@@
 		(dnp no)
 		(fields_autoplaced yes)
-		(property "Reference" "R21"
+		(property "Reference" "R23"
 			(at 73.66 41.91 90)
 			(show_name no)
@@
 			(project "at820_tiga"
 				(path "/a8c0f85c-55b6-4da9-ba8c-71a36ed08e24/3b744c5c-59b1-4c52-9315-8adf8de34fd5"
-					(reference "R21")
+					(reference "R23")
 					(unit 1)
 				)
@@
 		(dnp no)
 		(fields_autoplaced yes)
-		(property "Reference" "R23"
+		(property "Reference" "R25"
 			(at 127 133.3499 0)
 			(show_name no)
@@
 			(project "at820_tiga"
 				(path "/a8c0f85c-55b6-4da9-ba8c-71a36ed08e24/3b744c5c-59b1-4c52-9315-8adf8de34fd5"
-					(reference "R23")
+					(reference "R25")
 					(unit 1)
 				)
@@
 		(dnp no)
 		(fields_autoplaced yes)
-		(property "Reference" "R18"
+		(property "Reference" "R20"
 			(at 46.99 165.0999 0)
 			(show_name no)
@@
 			(project "at820_tiga"
 				(path "/a8c0f85c-55b6-4da9-ba8c-71a36ed08e24/3b744c5c-59b1-4c52-9315-8adf8de34fd5"
-					(reference "R18")
+					(reference "R20")
 					(unit 1)
 				)
@@
 		(dnp no)
 		(fields_autoplaced yes)
-		(property "Reference" "#PWR083"
+		(property "Reference" "#PWR084"
 			(at 34.29 78.74 0)
 			(hide yes)
@@
 			(project "at820_tiga"
 				(path "/a8c0f85c-55b6-4da9-ba8c-71a36ed08e24/3b744c5c-59b1-4c52-9315-8adf8de34fd5"
-					(reference "#PWR083")
+					(reference "#PWR084")
 					(unit 1)
 				)
