File: power.kicad_sch (KiCad schematic)
At the start: 38 parts, among them J10 QSPI_SWITCH, J8 USB_C_Receptacle_USB2.0_16P, J9 USB_C_Receptacle_USB2.0_16P, U4 AMS1117-3.3

Commit message: beta 2, modify board size, add some silkscreen
Parts:
- J10: renamed from J9; value USB_C_Receptacle_USB2.0_16P -> USB
- J9: renamed from J8; value USB_C_Receptacle_USB2.0_16P -> UART
- renumbered C15 to C16, C16 to C17, C17 to C18, C18 to C19, C19 to C20, C20 to C21, C21 to C22, C22 to C23, C23 to C24, C24 to C25, C25 to C26, C26 to C27, D1 to D10, D3 to D11, D6 to D3, D9 to D4, D7 to D5, D5 to D6, D8 to D7, D10 to D8, D2 to D9, H3 to H2, H2 to H3, J10 to J11, R13 to R10, R9 to R11, R10 to R12, R12 to R13, R11 to R14, R14 to R15, R7 to R8, R8 to R9

Commit message: v2 done
Parts:
- J11: value QSPI_SWITCH -> QSPI
- renumbered R8 to R10, R9 to R11, R10 to R12, R11 to R13, R12 to R14, R13 to R15, R14 to R16, R15 to R17
